File: Capstone-board-v1/Capstone-board-v1.kicad_sch (KiCad schematic)
At the start: 5 parts, among them U1 LT1121CN8-PBF, U2 NE555P, U3 GY-521

Commit message: correct footprints
Parts:
- added J1, J2: Conn_01x20_Socket, Connector_PinSocket_1.00mm:PinSocket_1x20_P1.00mm_Vertical, symbol Connector:Conn_01x20_Socket
- A1: footprint Raspberry Pi:MODULE_SC0918 -> Nima_double1:Double_Connector
- S1: footprint SW_TS02-66-60-BK-160-LCR-D -> TS02-66-60-BK-100-LCR-D:SW_TS02-66-60-BK-160-LCR-D
- U1: footprint Connector_PinSocket_2.54mm:PinSocket_2x04_P2.54mm_Vertical_SMD -> Package_DIP:DIP-8_W7.62mm
Other:
- moved on the sheet: A1

Commit message: so far
Parts:
- removed A1: SC0918, Nima_double1:Double_Connector, symbol Raspberry_Pi_Pico_W_Kicad_Files:SC0918
- added U4: L7805, symbol Regulator_Linear:L7805
Other:
- moved on the sheet: J1
Changed lines of the file:
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@@
     )
   )
-  (symbol (lib_id "Connector:Conn_01x20_Socket") (at 200.66 85.09 0) (unit 1)
-    (in_bom yes) (on_board yes) (dnp no) (fields_autoplaced)
-    (property "Reference" "J1" (at 201.93 85.09 0)
-      (effects (font (size 1.27 1.27)) (justify left))
-    )
-    (property "Value" "Conn_01x20_Socket" (at 201.93 87.63 0)
-      (effects (font (size 1.27 1.27)) (justify left))
-    )
-    (property "Footprint" "Connector_PinSocket_1.00mm:PinSocket_1x20_P1.00mm_Vertical" (at 200.66 85.09 0)
-      (effects (font (size 1.27 1.27)) hide)
-    )
-    (property "Datasheet" "~" (at 200.66 85.09 0)
+  (symbol (lib_id "Connector:Conn_01x20_Socket") (at 154.94 87.63 0) (unit 1)
+    (in_bom yes) (on_board yes) (dnp no)
+    (property "Reference" "J1" (at 149.86 59.69 0)
+      (effects (font (size 1.27 1.27)) (justify left))
+    )
+    (property "Value" "Conn_01x20_Socket" (at 144.78 55.88 0)
+      (effects (font (size 1.27 1.27)) (justify left))
+    )
+    (property "Footprint" "Connector_PinSocket_1.00mm:PinSocket_1x20_P1.00mm_Vertical" (at 154.94 87.63 0)
+      (effects (font (size 1.27 1.27)) hide)
+    )
+    (property "Datasheet" "~" (at 154.94 87.63 0)
       (effects (font (size 1.27 1.27)) hide)
     )
@@
     )
   )
-  (symbol (lib_id "Raspberry_Pi_Pico_W_Kicad_Files:SC0918") (at 161.29 99.06 0) (unit 1)
-    (in_bom yes) (on_board yes) (dnp no) (fields_autoplaced)
-    (property "Reference" "A1" (at 161.29 45.72 0)
-      (effects (font (size 1.27 1.27)))
-    )
-    (property "Value" "SC0918" (at 161.29 48.26 0)
-      (effects (font (size 1.27 1.27)))
-    )
-    (property "Footprint" "Nima_double1:Double_Connector" (at 161.29 50.8 0)
-      (effects (font (size 1.27 1.27)))
-    )
-    (property "Datasheet" "https://datasheets.raspberrypi.com/picow/pico-w-datasheet.pdf" (at 134.62 148.59 0)
-      (effects (font (size 1.27 1.27)) (justify left bottom) hide)
-    )
-    (property "manufacturer" "Raspberry Pi" (at 161.29 53.34 0)
-      (effects (font (size 1.27 1.27)))
-    )
-    (property "P/N" "SC0918" (at 161.29 48.26 0)
-      (effects (font (size 1.27 1.27)) hide)
-    )
-    (property "PARTREV" "1.6" (at 161.29 50.8 0)
-      (effects (font (size 1.27 1.27)) hide)
-    )
-    (property "MAXIMUM_PACKAGE_HEIGHT" "3.73mm" (at 161.29 53.34 0)
+  (symbol (lib_id "Connector:Conn_01x20_Socket") (at 120.65 90.17 180) (unit 1)
+    (in_bom yes) (on_board yes) (dnp no)
+    (property "Reference" "J2" (at 121.285 59.69 0)
+      (effects (font (size 1.27 1.27)))
+    )
+    (property "Value" "Conn_01x20_Socket" (at 121.92 55.88 0)
+      (effects (font (size 1.27 1.27)))
+    )
+    (property "Footprint" "Connector_PinSocket_1.00mm:PinSocket_1x20_P1.00mm_Vertical" (at 120.65 90.17 0)
+      (effects (font (size 1.27 1.27)) hide)
+    )
+    (property "Datasheet" "~" (at 120.65 90.17 0)
       (effects (font (size 1.27 1.27)) hide)
     )
@@
     (pin "2")
     (pin "20")
-    (pin "21")
-    (pin "22")
-    (pin "23")
-    (pin "24")
-    (pin "25")
-    (pin "26")
-    (pin "27")
-    (pin "28")
-    (pin "29")
-    (pin "3")
-    (pin "30")
-    (pin "31")
-    (pin "32")
-    (pin "33")
-    (pin "34")
-    (pin "35")
-    (pin "36")
-    (pin "37")
-    (pin "38")
-    (pin "39")
-    (pin "4")
-    (pin "40")
+    (pin "3")
+    (pin "4")
     (pin "5")
     (pin "6")
@@
       (project "Capstone-board-v1"
         (path "/5a0b0107-0183-4094-a3d7-2a417dfae25a"
-          (reference "A1") (unit 1)
-        )
-      )
-    )
-  )
-  (symbol (lib_id "Connector:Conn_01x20_Socket") (at 120.65 90.17 180) (unit 1)
-    (in_bom yes) (on_board yes) (dnp no) (fields_autoplaced)
-    (property "Reference" "J2" (at 121.285 59.69 0)
-      (effects (font (size 1.27 1.27)))
-    )
-    (property "Value" "Conn_01x20_Socket" (at 121.285 62.23 0)
-      (effects (font (size 1.27 1.27)))
-    )
-    (property "Footprint" "Connector_PinSocket_1.00mm:PinSocket_1x20_P1.00mm_Vertical" (at 120.65 90.17 0)
-      (effects (font (size 1.27 1.27)) hide)
-    )
-    (property "Datasheet" "~" (at 120.65 90.17 0)
-      (effects (font (size 1.27 1.27)) hide)
-    )
-    (pin "1")
-    (pin "10")
-    (pin "11")
-    (pin "12")
-    (pin "13")
-    (pin "14")
-    (pin "15")
-    (pin "16")
-    (pin "17")
-    (pin "18")
-    (pin "19")
-    (pin "2")
-    (pin "20")
-    (pin "3")
-    (pin "4")
-    (pin "5")
-    (pin "6")
-    (pin "7")
-    (pin "8")
-    (pin "9")
-    (instances
-      (project "Capstone-board-v1"
-        (path "/5a0b0107-0183-4094-a3d7-2a417dfae25a"
           (reference "J2") (unit 1)
         )
       )
+    )
+  )
+  (symbol (lib_id "Regulator_Linear:L7805") (at 39.37 81.28 0) (unit 1)
+    (in_bom yes) (on_board yes) (dnp no) (fields_autoplaced)
+    (property "Reference" "U4" (at 39.37 74.93 0)
+      (effects (font (size 1.27 1.27)))
+    )
+    (property "Value" "L7805" (at 39.37 77.47 0)
+      (effects (font (size 1.27 1.27)))
+    )
+    (property "Footprint" "" (at 40.005 85.09 0)
+      (effects (font (size 1.27 1.27) italic) (justify left) hide)
+    )
+    (property "Datasheet" "http://www.st.com/content/ccc/resource/technical/document/datasheet/41/4f/b3/b0/12/d4/47/88/CD00000444.pdf/files/CD00000444.pdf/jcr:content/translations/en.CD00000444.pdf" (at 39.37 82.55 0)
+      (effects (font (size 1.27 1.27)) hide)
+    )
+    (pin "1")
+    (pin "2")
+    (pin "3")
+    (instances
+      (project "Capstone-board-v1"
+        (path "/5a0b0107-0183-4094-a3d7-2a417dfae25a"
+          (reference "U4") (unit 1)
+        )
+      )
