File: Capstone-board-v1/Capstone-board-car.kicad_sch (KiCad schematic)
At the start: 22 parts, among them J1 Pico Socket 1, J2 Pico Socket 2, M1 DC Vibration Motor, Q1 2N3904, U1 3.3 V Voltage Regulator, U2 555 Timer, U3 Gyroscope Sensor, U4 OP-Amp, U5 Hall Effect Sensor

Commit message: schematic
Parts:
- removed D2: 1N4001, Diode_THT:D_DO-41_SOD81_P10.16mm_Horizontal, symbol Diode:1N4001
- removed M1: DC Vibration Motor, symbol Motor:Motor_DC
- removed Q1: 2N3904, Package_TO_SOT_THT:TO-92_Inline, symbol Transistor_BJT:2N3904
- removed U3: Gyroscope Sensor, GY-521:GY-521, symbol GY-521:GY-521
- removed U4: OP-Amp, symbol Amplifier_Operational:TLV2372
- removed U5: Hall Effect Sensor, Sensor_Current:Allegro_SIP-4, symbol Sensor_Current:A1363xKTTN-1
- added BT2: Battery, symbol Device:Battery
- added C4, C6: 0.1uF, symbol Device:C
- added C5: 0.47uF, symbol Device:C
- added J3: Ultra Sonic Sensor, symbol Connector:Conn_01x04_Socket
- added J4: Car, symbol Connector:Conn_01x08_Socket
- added J5: Camera, symbol Connector:Conn_01x02_Socket
- added U3: 5V Voltage Regulator 2, symbol Regulator_Linear:L7805
- added U4: 5V Voltage Regulator 1, symbol Regulator_Linear:L7805
- C3: value 0.1uF -> 0.47uF
- J1: value Pico Socket 1 -> Pcio Socket 1
- R1: value 100kOhms -> 100KOhms
- R4: value 1KOhms -> 270Ohms
- R5: value 1KOhms -> 10Ohms
- R6: value 5.6KOhms -> 10Ohms
- S1: value Pushbutton -> Push Button
- U1: value 3.3 V Voltage Regulator -> 3.3V Voltage Regulator
Connections:
- net Earth: now also C3.2, R4.1, R5.1, R6.1, BT2.2 (-), C4.2, C5.2, C6.2, J3.4 (Pin_4), J4.2 (Pin_2), J5.2 (Pin_2), U3.2 (GND), U4.2 (GND); no longer R5.2
- net VCC: now also C3.1, R3.2, U4.1 (IN)
- net at U2.2 (TR), U2.6 (THR): now also R2.2, R3.1, S1.4; no longer R3.2
- net at J1.2 (Pin_2): now also J4.4 (Pin_4)
- net at J1.1 (Pin_1): now also J4.3 (Pin_3)
- net at C2.1, J2.19 (Pin_19), U1.1 (OUT): no longer C3.1
- net at R4.2: now also C4.1, J3.1 (Pin_1), U4.3 (OUT); no longer J1.17 (Pin_17)
- net at J1.20 (Pin_20): now also J3.2 (Pin_2); no longer R6.1
- net at R6.2: now also R5.2, C6.1, J5.1 (Pin_1), U3.3 (OUT); no longer R5.1
- net at J1.19 (Pin_19): now also J3.3 (Pin_3)
- net at J1.4 (Pin_4): now also J4.5 (Pin_5)
- net at J1.5 (Pin_5): now also J4.6 (Pin_6)
- net at J1.6 (Pin_6): now also J4.7 (Pin_7)
- net at J1.7 (Pin_7): now also J4.8 (Pin_8)
- new net VCCQ: BT2.1 (+), C5.1, J4.1 (Pin_1), U3.1 (IN)
Other:
- note added: "Car PCB"
- note removed: "Glove PCB"
- moved on the sheet: BT1, C1, C2, D1, J1, J2, R1, R2, R3, S1, U1, U2

Commit message: ready for tracing
Parts:
- BT1, BT2: footprint (none) -> Battery:Battery_Panasonic_CR1025-VSK_Vertical_CircularHoles
- C1, C2, C3, C4, C5, C6: footprint (none) -> Capacitor_THT:CP_Axial_L10.0mm_D4.5mm_P15.00mm_Horizontal
- J3: footprint (none) -> Connector_PinHeader_1.27mm:PinHeader_1x04_P1.27mm_Vertical
- J4: footprint (none) -> Connector_PinHeader_1.27mm:PinHeader_1x08_P1.27mm_Vertical
- J5: footprint (none) -> Connector_PinHeader_1.27mm:PinHeader_1x02_P1.27mm_Vertical
- R1, R2, R3, R4, R5, R6: footprint (none) -> Resistor_THT:R_Axial_DIN0204_L3.6mm_D1.6mm_P1.90mm_Vertical
- U3, U4: footprint (none) -> Package_DIP:DIP-8_W7.62mm_Socket
Changed lines of the file:
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@@
       (effects (font (size 1.27 1.27)) (justify right))
     )
-    (property "Footprint" "" (at 95.504 168.656 90)
+    (property "Footprint" "Resistor_THT:R_Axial_DIN0204_L3.6mm_D1.6mm_P1.90mm_Vertical" (at 95.504 168.656 90)
       (effects (font (size 1.27 1.27)) hide)
     )
@@
       (effects (font (size 1.27 1.27)) (justify left))
     )
-    (property "Footprint" "" (at 83.5152 135.89 0)
+    (property "Footprint" "Capacitor_THT:CP_Axial_L10.0mm_D4.5mm_P15.00mm_Horizontal" (at 83.5152 135.89 0)
       (effects (font (size 1.27 1.27)) hide)
     )
@@
       (effects (font (size 1.27 1.27)))
     )
-    (property "Footprint" "" (at 71.755 165.1 0)
+    (property "Footprint" "Package_DIP:DIP-8_W7.62mm_Socket" (at 71.755 165.1 0)
       (effects (font (size 1.27 1.27) italic) (justify left) hide)
     )
@@
       (effects (font (size 1.27 1.27)) (justify right))
     )
-    (property "Footprint" "" (at 89.154 102.616 90)
+    (property "Footprint" "Resistor_THT:R_Axial_DIN0204_L3.6mm_D1.6mm_P1.90mm_Vertical" (at 89.154 102.616 90)
       (effects (font (size 1.27 1.27)) hide)
     )
@@
       (effects (font (size 1.27 1.27)) (justify left))
     )
-    (property "Footprint" "" (at 50.8 53.086 90)
+    (property "Footprint" "Battery:Battery_Panasonic_CR1025-VSK_Vertical_CircularHoles" (at 50.8 53.086 90)
       (effects (font (size 1.27 1.27)) hide)
     )
@@
       (effects (font (size 1.27 1.27)))
     )
-    (property "Footprint" "" (at 236.22 125.73 0)
+    (property "Footprint" "Connector_PinHeader_1.27mm:PinHeader_1x08_P1.27mm_Vertical" (at 236.22 125.73 0)
       (effects (font (size 1.27 1.27)) hide)
     )
@@
       (effects (font (size 1.27 1.27)) (justify left))
     )
-    (property "Footprint" "" (at 83.5152 172.72 0)
+    (property "Footprint" "Capacitor_THT:CP_Axial_L10.0mm_D4.5mm_P15.00mm_Horizontal" (at 83.5152 172.72 0)
       (effects (font (size 1.27 1.27)) hide)
     )
@@
       (effects (font (size 1.27 1.27)) (justify right))
     )
-    (property "Footprint" "" (at 96.774 131.826 90)
+    (property "Footprint" "Resistor_THT:R_Axial_DIN0204_L3.6mm_D1.6mm_P1.90mm_Vertical" (at 96.774 131.826 90)
       (effects (font (size 1.27 1.27)) hide)
     )
@@
       (effects (font (size 1.27 1.27)) (justify left))
     )
-    (property "Footprint" "" (at 36.83 53.086 90)
+    (property "Footprint" "Battery:Battery_Panasonic_CR1025-VSK_Vertical_CircularHoles" (at 36.83 53.086 90)
       (effects (font (size 1.27 1.27)) hide)
     )
@@
       (effects (font (size 1.27 1.27)) (justify right))
     )
-    (property "Footprint" "" (at 89.154 92.456 90)
+    (property "Footprint" "Resistor_THT:R_Axial_DIN0204_L3.6mm_D1.6mm_P1.90mm_Vertical" (at 89.154 92.456 90)
       (effects (font (size 1.27 1.27)) hide)
     )
@@
       (effects (font (size 1.27 1.27)))
     )
-    (property "Footprint" "" (at 95.504 85.344 90)
+    (property "Footprint" "Resistor_THT:R_Axial_DIN0204_L3.6mm_D1.6mm_P1.90mm_Vertical" (at 95.504 85.344 90)
       (effects (font (size 1.27 1.27)) hide)
     )
@@
       (effects (font (size 1.27 1.27)) (justify left))
     )
-    (property "Footprint" "" (at 60.6552 172.72 0)
+    (property "Footprint" "Capacitor_THT:CP_Axial_L10.0mm_D4.5mm_P15.00mm_Horizontal" (at 60.6552 172.72 0)
       (effects (font (size 1.27 1.27)) hide)
     )
@@
       (effects (font (size 1.27 1.27)) (justify left))
     )
-    (property "Footprint" "" (at 60.6552 135.89 0)
+    (property "Footprint" "Capacitor_THT:CP_Axial_L10.0mm_D4.5mm_P15.00mm_Horizontal" (at 60.6552 135.89 0)
       (effects (font (size 1.27 1.27)) hide)
     )
@@
       (effects (font (size 1.27 1.27)) (justify right))
     )
-    (property "Footprint" "" (at 109.474 168.656 90)
+    (property "Footprint" "Resistor_THT:R_Axial_DIN0204_L3.6mm_D1.6mm_P1.90mm_Vertical" (at 109.474 168.656 90)
       (effects (font (size 1.27 1.27)) hide)
     )
@@
       (effects (font (size 1.27 1.27)))
     )
-    (property "Footprint" "" (at 137.16 127 0)
+    (property "Footprint" "Connector_PinHeader_1.27mm:PinHeader_1x04_P1.27mm_Vertical" (at 137.16 127 0)
       (effects (font (size 1.27 1.27)) hide)
     )
@@
       (effects (font (size 1.27 1.27)) (justify left))
     )
-    (property "Footprint" "" (at 132.08 167.64 0)
+    (property "Footprint" "Connector_PinHeader_1.27mm:PinHeader_1x02_P1.27mm_Vertical" (at 132.08 167.64 0)
       (effects (font (size 1.27 1.27)) hide)
     )
@@
       (effects (font (size 1.27 1.27)) (justify left))
     )
-    (property "Footprint" "" (at 148.2852 80.01 0)
+    (property "Footprint" "Capacitor_THT:CP_Axial_L10.0mm_D4.5mm_P15.00mm_Horizontal" (at 148.2852 80.01 0)
       (effects (font (size 1.27 1.27)) hide)
     )
@@
       (effects (font (size 1.27 1.27)) (justify left))
     )
-    (property "Footprint" "" (at 54.3052 97.79 0)
+    (property "Footprint" "Capacitor_THT:CP_Axial_L10.0mm_D4.5mm_P15.00mm_Horizontal" (at 54.3052 97.79 0)
       (effects (font (size 1.27 1.27)) hide)
     )
@@
       (effects (font (size 1.27 1.27)))
     )
-    (property "Footprint" "" (at 71.755 128.27 0)
+    (property "Footprint" "Package_DIP:DIP-8_W7.62mm_Socket" (at 71.755 128.27 0)
       (effects (font (size 1.27 1.27) italic) (justify left) hide)
     )

Commit message: correct hole size
Parts:
- C1, C2, C3, C4, C5, C6: footprint Capacitor_THT:CP_Axial_L10.0mm_D4.5mm_P15.00mm_Horizontal -> Capacitor_THT:CP_Radial_Tantal_D4.5mm_P5.00mm
- J1, J2: footprint Connector_PinSocket_1.00mm:PinSocket_1x20_P1.00mm_Vertical -> Connector_PinSocket_2.54mm:PinSocket_1x20_P2.54mm_Vertical
- J3: footprint Connector_PinHeader_1.27mm:PinHeader_1x04_P1.27mm_Vertical -> Connector_PinHeader_2.54mm:PinHeader_1x04_P2.54mm_Vertical
- J4: footprint Connector_PinHeader_1.27mm:PinHeader_1x08_P1.27mm_Vertical -> Connector_PinHeader_2.54mm:PinHeader_1x08_P2.54mm_Vertical
- J5: footprint Connector_PinHeader_1.27mm:PinHeader_1x02_P1.27mm_Vertical -> Connector_PinHeader_2.54mm:PinHeader_1x02_P2.54mm_Vertical
- R1, R2, R3, R4, R5, R6: footprint Resistor_THT:R_Axial_DIN0204_L3.6mm_D1.6mm_P1.90mm_Vertical -> Resistor_THT:R_Axial_DIN0204_L3.6mm_D1.6mm_P5.08mm_Horizontal
- U3, U4: footprint Package_DIP:DIP-8_W7.62mm_Socket -> LinReg:TO255P1040X460X1968-3
Changed lines of the file:
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@@
       (effects (font (size 1.27 1.27)) (justify right))
     )
-    (property "Footprint" "Resistor_THT:R_Axial_DIN0204_L3.6mm_D1.6mm_P1.90mm_Vertical" (at 95.504 168.656 90)
+    (property "Footprint" "Resistor_THT:R_Axial_DIN0204_L3.6mm_D1.6mm_P5.08mm_Horizontal" (at 95.504 168.656 90)
       (effects (font (size 1.27 1.27)) hide)
     )
@@
       (effects (font (size 1.27 1.27)) (justify left))
     )
-    (property "Footprint" "Capacitor_THT:CP_Axial_L10.0mm_D4.5mm_P15.00mm_Horizontal" (at 83.5152 135.89 0)
+    (property "Footprint" "Capacitor_THT:CP_Radial_Tantal_D4.5mm_P5.00mm" (at 83.5152 135.89 0)
       (effects (font (size 1.27 1.27)) hide)
     )
@@
       (effects (font (size 1.27 1.27)))
     )
-    (property "Footprint" "Package_DIP:DIP-8_W7.62mm_Socket" (at 71.755 165.1 0)
+    (property "Footprint" "LinReg:TO255P1040X460X1968-3" (at 71.755 165.1 0)
       (effects (font (size 1.27 1.27) italic) (justify left) hide)
     )
@@
       (effects (font (size 1.27 1.27)) (justify right))
     )
-    (property "Footprint" "Resistor_THT:R_Axial_DIN0204_L3.6mm_D1.6mm_P1.90mm_Vertical" (at 89.154 102.616 90)
+    (property "Footprint" "Resistor_THT:R_Axial_DIN0204_L3.6mm_D1.6mm_P5.08mm_Horizontal" (at 89.154 102.616 90)
       (effects (font (size 1.27 1.27)) hide)
     )
@@
       (effects (font (size 1.27 1.27)))
     )
-    (property "Footprint" "Connector_PinHeader_1.27mm:PinHeader_1x08_P1.27mm_Vertical" (at 236.22 125.73 0)
+    (property "Footprint" "Connector_PinHeader_2.54mm:PinHeader_1x08_P2.54mm_Vertical" (at 236.22 125.73 0)
       (effects (font (size 1.27 1.27)) hide)
     )
@@
       (effects (font (size 1.27 1.27)) (justify left))
     )
-    (property "Footprint" "Capacitor_THT:CP_Axial_L10.0mm_D4.5mm_P15.00mm_Horizontal" (at 83.5152 172.72 0)
+    (property "Footprint" "Capacitor_THT:CP_Radial_Tantal_D4.5mm_P5.00mm" (at 83.5152 172.72 0)
       (effects (font (size 1.27 1.27)) hide)
     )
@@
       (effects (font (size 1.27 1.27)) (justify right))
     )
-    (property "Footprint" "Resistor_THT:R_Axial_DIN0204_L3.6mm_D1.6mm_P1.90mm_Vertical" (at 96.774 131.826 90)
+    (property "Footprint" "Resistor_THT:R_Axial_DIN0204_L3.6mm_D1.6mm_P5.08mm_Horizontal" (at 96.774 131.826 90)
       (effects (font (size 1.27 1.27)) hide)
     )
@@
       (effects (font (size 1.27 1.27)) (justify right))
     )
-    (property "Footprint" "Resistor_THT:R_Axial_DIN0204_L3.6mm_D1.6mm_P1.90mm_Vertical" (at 89.154 92.456 90)
+    (property "Footprint" "Resistor_THT:R_Axial_DIN0204_L3.6mm_D1.6mm_P5.08mm_Horizontal" (at 89.154 92.456 90)
       (effects (font (size 1.27 1.27)) hide)
     )
@@
       (effects (font (size 1.27 1.27)))
     )
-    (property "Footprint" "Resistor_THT:R_Axial_DIN0204_L3.6mm_D1.6mm_P1.90mm_Vertical" (at 95.504 85.344 90)
+    (property "Footprint" "Resistor_THT:R_Axial_DIN0204_L3.6mm_D1.6mm_P5.08mm_Horizontal" (at 95.504 85.344 90)
       (effects (font (size 1.27 1.27)) hide)
     )
@@
       (effects (font (size 1.27 1.27)) (justify left))
     )
-    (property "Footprint" "Capacitor_THT:CP_Axial_L10.0mm_D4.5mm_P15.00mm_Horizontal" (at 60.6552 172.72 0)
+    (property "Footprint" "Capacitor_THT:CP_Radial_Tantal_D4.5mm_P5.00mm" (at 60.6552 172.72 0)
       (effects (font (size 1.27 1.27)) hide)
     )
@@
       (effects (font (size 1.27 1.27)) (justify left))
     )
-    (property "Footprint" "Capacitor_THT:CP_Axial_L10.0mm_D4.5mm_P15.00mm_Horizontal" (at 60.6552 135.89 0)
+    (property "Footprint" "Capacitor_THT:CP_Radial_Tantal_D4.5mm_P5.00mm" (at 60.6552 135.89 0)
       (effects (font (size 1.27 1.27)) hide)
     )
@@
       (effects (font (size 1.27 1.27)) (justify left))
     )
-    (property "Footprint" "Connector_PinSocket_1.00mm:PinSocket_1x20_P1.00mm_Vertical" (at 238.76 78.74 0)
+    (property "Footprint" "Connector_PinSocket_2.54mm:PinSocket_1x20_P2.54mm_Vertical" (at 238.76 78.74 0)
       (effects (font (size 1.27 1.27)) hide)
     )
@@
       (effects (font (size 1.27 1.27)) (justify right))
     )
-    (property "Footprint" "Resistor_THT:R_Axial_DIN0204_L3.6mm_D1.6mm_P1.90mm_Vertical" (at 109.474 168.656 90)
+    (property "Footprint" "Resistor_THT:R_Axial_DIN0204_L3.6mm_D1.6mm_P5.08mm_Horizontal" (at 109.474 168.656 90)
       (effects (font (size 1.27 1.27)) hide)
     )
@@
       (effects (font (size 1.27 1.27)))
     )
-    (property "Footprint" "Connector_PinSocket_1.00mm:PinSocket_1x20_P1.00mm_Vertical" (at 256.54 81.28 0)
+    (property "Footprint" "Connector_PinSocket_2.54mm:PinSocket_1x20_P2.54mm_Vertical" (at 256.54 81.28 0)
       (effects (font (size 1.27 1.27)) hide)
     )
@@
       (effects (font (size 1.27 1.27)))
     )
-    (property "Footprint" "Connector_PinHeader_1.27mm:PinHeader_1x04_P1.27mm_Vertical" (at 137.16 127 0)
+    (property "Footprint" "Connector_PinHeader_2.54mm:PinHeader_1x04_P2.54mm_Vertical" (at 137.16 127 0)
       (effects (font (size 1.27 1.27)) hide)
     )
@@
       (effects (font (size 1.27 1.27)) (justify left))
     )
-    (property "Footprint" "Connector_PinHeader_1.27mm:PinHeader_1x02_P1.27mm_Vertical" (at 132.08 167.64 0)
+    (property "Footprint" "Connector_PinHeader_2.54mm:PinHeader_1x02_P2.54mm_Vertical" (at 132.08 167.64 0)
       (effects (font (size 1.27 1.27)) hide)
     )
@@
       (effects (font (size 1.27 1.27)) (justify left))
     )
-    (property "Footprint" "Capacitor_THT:CP_Axial_L10.0mm_D4.5mm_P15.00mm_Horizontal" (at 148.2852 80.01 0)
+    (property "Footprint" "Capacitor_THT:CP_Radial_Tantal_D4.5mm_P5.00mm" (at 148.2852 80.01 0)
       (effects (font (size 1.27 1.27)) hide)
     )
@@
       (effects (font (size 1.27 1.27)) (justify left))
     )
-    (property "Footprint" "Capacitor_THT:CP_Axial_L10.0mm_D4.5mm_P15.00mm_Horizontal" (at 54.3052 97.79 0)
+    (property "Footprint" "Capacitor_THT:CP_Radial_Tantal_D4.5mm_P5.00mm" (at 54.3052 97.79 0)
       (effects (font (size 1.27 1.27)) hide)
     )
@@
       (effects (font (size 1.27 1.27)))
     )
-    (property "Footprint" "Package_DIP:DIP-8_W7.62mm_Socket" (at 71.755 128.27 0)
+    (property "Footprint" "LinReg:TO255P1040X460X1968-3" (at 71.755 128.27 0)
       (effects (font (size 1.27 1.27) italic) (justify left) hide)
     )
