File: Capstone-board-v1/Capstone-board-car.kicad_sch (KiCad schematic)
At the start: 25 parts, among them J1 Pico Socket 1, J2 Pico Socket 2, J3 Ultra Sonic Sensor, J4 Car, J5 Camera, J6 Gyroscope Sensor, U1 3.3V V.R, U2 555 Timer, U3 5V V.R 2, U4 5V V.R 1

Commit message: Final PCB's done.
Connections:
- net VCC: no longer C3.1, U4.1 (IN)
- net at R1.2, U1.8 (IN), U2.3 (Q): now also C3.1, U4.1 (IN)
Changed lines of the file:
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@@
   (junction (at 59.69 161.29) (diameter 0) (color 0 0 0 0)
   )
+  (junction (at 134.62 86.36) (diameter 0) (color 0 0 0 0)
+  )
   (junction (at 227.33 139.7) (diameter 0) (color 0 0 0 0)
   )
@@
     (stroke (width 0) (type default))
   )
+  (wire (pts (xy 134.62 96.52) (xy 134.62 86.36))
+    (stroke (width 0) (type default))
+  )
   (wire (pts (xy 219.71 133.35) (xy 231.14 133.35))
     (stroke (width 0) (type default))
@@
     (stroke (width 0) (type default))
   )
+  (wire (pts (xy 116.84 96.52) (xy 134.62 96.52))
+    (stroke (width 0) (type default))
+  )
   (wire (pts (xy 124.46 167.64) (xy 127 167.64))
     (stroke (width 0) (type default))
@@
     (stroke (width 0) (type default))
   )
-  (wire (pts (xy 53.34 124.46) (xy 53.34 119.38))
+  (wire (pts (xy 53.34 114.3) (xy 53.34 124.46))
     (stroke (width 0) (type default))
   )
@@
     (stroke (width 0) (type default))
   )
+  (wire (pts (xy 53.34 114.3) (xy 116.84 114.3))
+    (stroke (width 0) (type default))
+  )
   (wire (pts (xy 132.08 127) (xy 129.54 127))
     (stroke (width 0) (type default))
@@
   )
   (wire (pts (xy 71.12 138.43) (xy 71.12 142.24))
+    (stroke (width 0) (type default))
+  )
+  (wire (pts (xy 116.84 114.3) (xy 116.84 96.52))
     (stroke (width 0) (type default))
   )
@@
         )
       )
-    )
-  )
-  (symbol (lib_id "power:VCC") (at 53.34 119.38 0) (unit 1)
-    (in_bom yes) (on_board yes) (dnp no) (fields_autoplaced)
-    (property "Reference" "#PWR08" (at 53.34 123.19 0)
-      (effects (font (size 1.27 1.27)) hide)
-    )
-    (property "Value" "VCC" (at 53.34 114.3 0)
-      (effects (font (size 1.27 1.27)))
-    )
-    (property "Footprint" "" (at 53.34 119.38 0)
-      (effects (font (size 1.27 1.27)) hide)
-    )
-    (property "Datasheet" "" (at 53.34 119.38 0)
-      (effects (font (size 1.27 1.27)) hide)
-    )
-    (pin "1")
-    (instances
-      (project "Capstone-board-car"
-        (path "/5a0b0107-0183-4094-a3d7-2a417dfae25a"
-          (reference "#PWR08") (unit 1)
-        )
-      )

Commit message: Final PCBs done!
Parts:
- removed R4, R5, R6: 10Ohms, Resistor_THT:R_Axial_DIN0204_L3.6mm_D1.6mm_P5.08mm_Horizontal, symbol Device:R_US
- added J7: Compass, Connector_PinSocket_2.54mm:PinSocket_1x05_P2.54mm_Vertical, symbol Connector:Conn_01x05_Socket
- BT1: footprint Connector_Hirose:Hirose_DF11-4DP-2DSA_2x02_P2.00mm_Vertical -> Connector_Hirose:Hirose_DF11-6DP-2DSA_2x03_P2.00mm_Vertical
- J4: value Car -> Car Motor 1
- J6: value Gyroscope Sensor -> Car Motor 2
- U3: value 5V V.R 2 -> 5V Buck Conv
- U4: value 5V V.R 1 -> 5V V.R
Connections:
- net Earth: now also J7.2 (Pin_2)
- net VCCQ: now also J6.1 (Pin_1)
- net at J1.15 (Pin_15): now also J7.5 (Pin_5)
- net at J1.16 (Pin_16): now also J7.4 (Pin_4)
- net at J1.17 (Pin_17): now also J7.3 (Pin_3)
- net at C2.1, J2.19 (Pin_19), U1.1 (OUT): now also J7.1 (Pin_1); no longer J6.1 (Pin_1)
- net at J2.1 (Pin_1): no longer J6.4 (Pin_4)
- net at J2.11 (Pin_11): now also J6.5 (Pin_5)
- net at J2.12 (Pin_12): now also J6.4 (Pin_4)
- net at J2.14 (Pin_14): now also J6.3 (Pin_3)
- net at J2.2 (Pin_2): no longer J6.3 (Pin_3)
- net at J2.6 (Pin_6): now also J6.8 (Pin_8)
- net at J2.7 (Pin_7): now also J6.7 (Pin_7)
- net at J2.9 (Pin_9): now also J6.6 (Pin_6)
