File: Capstone-board-v1/Capstone-board-v1.kicad_pcb (KiCad board)
At the start: 2 copper layers, 53.9 x 47.3 mm, 21 parts, among them J1 Pico Socket 1, J2 Pico Socket 2, J3 Gyroscope Sensor, M1 DC Vibration Motor, Q1 2N3904, U1 3.3 V V.R, U2 555 Timer, U3 Hall Effect Sensor, U4 OP Amp

Commit message: Final PCBs done!
Parts:
- BT1: footprint Connector_Hirose:Hirose_DF11-4DP-2DSA_2x02_P2.00mm_Vertical -> Connector_Hirose:Hirose_DF11-6DP-2DSA_2x03_P2.00mm_Vertical
- M1: footprint Connector_Hirose:Hirose_DF13-02P-1.25DSA_1x02_P1.25mm_Vertical -> Connector_PinSocket_2.54mm:PinSocket_1x02_P2.54mm_Vertical
- U3: footprint Connector_Hirose:Hirose_DF13-03P-1.25DSA_1x03_P1.25mm_Vertical -> Connector_PinSocket_2.54mm:PinSocket_1x03_P2.54mm_Vertical
- moved U3 2.92 mm to (27.1, 23.5), turned to 90 degrees
- moved BT1 2.13 mm to (54.7, 59.6)
- moved M1 0.73 mm to (44.9, 23.5), turned to 90 degrees
Routing:
- net Earth: track 193.9 -> 202.5 mm
- net Net-(U1-IN): track 98.5 -> 92.1 mm
- net Net-(U3-VOUT): track 40.8 -> 37.9 mm
- net VCC: track 31.6 -> 30.0 mm
- net Net-(D1-A): track 53.9 -> 52.8 mm
Other:
- board size 53.9 x 47.3 mm -> 54.4 x 47.6 mm
- board text added: "M1"
- board text added: "U3"
